File: hardware/firepot-loadcells/firepot-loadcells.kicad_sch (KiCad schematic)
At the start: 17 parts, among them U1 HX711, U2 HX711, U3 HX711, U4 HX711, U5 HX711, U6 HX711, U7 HX711, U8 HX711, U9 XIAO ESP32S3

Commit message: Redraw the load cell schematic flat
Landscape A3, four columns, one row per island. Each load cell sits
hard against its HX711 with the four output pins landing on the input
pins, so there is no wire between them. Every board-to-board net is a
named label now: 3V3, GND, SCK, and one BINn_DT line per cell. The
long bus lines down the old portrait sheet are gone. Netlist and ERC
unchanged.

Co-Authored-By: Claude Sonnet 5 <noreply@anthropic.com>
Other:
- note added: "D3 to D6 read the left island, bins 0, 1, 4, 5. D7 to D10 read the right island, bins 2, 3, 6, 7."
- note added: "Every board-to-board net is a named label: 3V3, GND, SCK, and one BINn_DT data line per cell."
- note added: "Load cell wire colours: red E+, black E-, green A+, white A-. Check them against your own cell."
- note added: "VCC and VDD are shorted at every HX711. Both go to 3V3."
- note removed: "Check them against your own cell."
- note removed: "D3 to D6 serve the left island, D7 to D10 the right. Crossing wires join only at a dot."
- note removed: "Load cell wire colours: red E+, black E-, green A+, white A-."
- note removed: "VCC and VDD are shorted at every HX711. Board-to-board runs use screw terminals."

Commit message: Tighten and darken the load cell schematic
Export in black and white with no drawing sheet, so it reads as solid
black on white instead of the pale KiCad pastels. Sheet shrunk to fit
the drawing, text up to 3.5 mm, XIAO body widened so its pin names
stop colliding. Same four-column flat layout, same netlist.

Co-Authored-By: Claude Sonnet 5 <noreply@anthropic.com>
Parts:
- LC1: value bin 0, far left -> Bin 0
- LC2: value bin 1, far centre-left -> Bin 1
- LC3: value bin 4, near left -> Bin 4
- LC4: value bin 5, near centre-left -> Bin 5
- LC5: value bin 7, near right -> Bin 7
- LC6: value bin 6, near centre-right -> Bin 6
- LC7: value bin 3, far right -> Bin 3
- LC8: value bin 2, far centre-right -> Bin 2
Other:
- note added: "3V3, GND, SCK and the eight BINn_DT data lines are the only board-to-board nets. Each one is a named label."
- note added: "Load cell wires: red E+, black E-, green A+, white A-. Check against your own cell."
- note added: "The grid matches the table: far row bins 0 to 3, near row bins 4 to 7. D3 to D6 read the left island, D7 to D10 the right."
- note added: "VCC and VDD are shorted at each HX711 and both go to 3V3."
- note removed: "3V3, GND and SCK are split 1-to-4 by a PCT-215 lever connector per rail, per island."
- note removed: "D3 to D6 read the left island, bins 0, 1, 4, 5. D7 to D10 read the right island, bins 2, 3, 6, 7."
- note removed: "Every board-to-board net is a named label: 3V3, GND, SCK, and one BINn_DT data line per cell."
- note removed: "Load cell wire colours: red E+, black E-, green A+, white A-. Check them against your own cell."
- note removed: "VCC and VDD are shorted at every HX711. Both go to 3V3."

Commit message: Drop the label flags, keep the net names
Every BINn_DT and USB net was a global label, which KiCad draws as a
tag shape that collided with its neighbours. They are plain sheet
labels now: just the net name on the wire end. Netlist unchanged.

Co-Authored-By: Claude Sonnet 5 <noreply@anthropic.com>
Changed lines of the file:
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@@
 		(stroke (width 0.254) (type default))
 	)
-	(global_label "BIN0_DT" (shape output) (at 68.58 17.78 0)
-		(effects (font (size 3.5 3.5)) (justify left))
-		(property "Intersheetrefs" "${INTERSHEET_REFS}" (at 68.58 17.78 0)
-			(effects (font (size 1.27 1.27)) (hide yes))
-		)
+	(label "BIN0_DT" (at 68.58 17.78 0)
+		(effects (font (size 3.5 3.5)) (justify left))
 	)
 	(wire (pts (xy 63.5 22.86) (xy 68.58 22.86))
@@
 		(stroke (width 0.254) (type default))
 	)
-	(global_label "BIN1_DT" (shape output) (at 154.94 17.78 0)
-		(effects (font (size 3.5 3.5)) (justify left))
-		(property "Intersheetrefs" "${INTERSHEET_REFS}" (at 154.94 17.78 0)
-			(effects (font (size 1.27 1.27)) (hide yes))
-		)
+	(label "BIN1_DT" (at 154.94 17.78 0)
+		(effects (font (size 3.5 3.5)) (justify left))
 	)
 	(wire (pts (xy 149.86 22.86) (xy 154.94 22.86))
@@
 		(stroke (width 0.254) (type default))
 	)
-	(global_label "BIN2_DT" (shape output) (at 241.3 17.78 0)
-		(effects (font (size 3.5 3.5)) (justify left))
-		(property "Intersheetrefs" "${INTERSHEET_REFS}" (at 241.3 17.78 0)
-			(effects (font (size 1.27 1.27)) (hide yes))
-		)
+	(label "BIN2_DT" (at 241.3 17.78 0)
+		(effects (font (size 3.5 3.5)) (justify left))
 	)
 	(wire (pts (xy 236.22 22.86) (xy 241.3 22.86))
@@
 		(stroke (width 0.254) (type default))
 	)
-	(global_label "BIN3_DT" (shape output) (at 327.66 17.78 0)
-		(effects (font (size 3.5 3.5)) (justify left))
-		(property "Intersheetrefs" "${INTERSHEET_REFS}" (at 327.66 17.78 0)
-			(effects (font (size 1.27 1.27)) (hide yes))
-		)
+	(label "BIN3_DT" (at 327.66 17.78 0)
+		(effects (font (size 3.5 3.5)) (justify left))
 	)
 	(wire (pts (xy 322.58 22.86) (xy 327.66 22.86))
@@
 		(stroke (width 0.254) (type default))
 	)
-	(global_label "BIN4_DT" (shape output) (at 68.58 58.42 0)
-		(effects (font (size 3.5 3.5)) (justify left))
-		(property "Intersheetrefs" "${INTERSHEET_REFS}" (at 68.58 58.42 0)
-			(effects (font (size 1.27 1.27)) (hide yes))
-		)
+	(label "BIN4_DT" (at 68.58 58.42 0)
+		(effects (font (size 3.5 3.5)) (justify left))
 	)
 	(wire (pts (xy 63.5 63.5) (xy 68.58 63.5))
@@
 		(stroke (width 0.254) (type default))
 	)
-	(global_label "BIN5_DT" (shape output) (at 154.94 58.42 0)
-		(effects (font (size 3.5 3.5)) (justify left))
-		(property "Intersheetrefs" "${INTERSHEET_REFS}" (at 154.94 58.42 0)
-			(effects (font (size 1.27 1.27)) (hide yes))
-		)
+	(label "BIN5_DT" (at 154.94 58.42 0)
+		(effects (font (size 3.5 3.5)) (justify left))
 	)
 	(wire (pts (xy 149.86 63.5) (xy 154.94 63.5))
@@
 		(stroke (width 0.254) (type default))
 	)
-	(global_label "BIN6_DT" (shape output) (at 241.3 58.42 0)
-		(effects (font (size 3.5 3.5)) (justify left))
-		(property "Intersheetrefs" "${INTERSHEET_REFS}" (at 241.3 58.42 0)
-			(effects (font (size 1.27 1.27)) (hide yes))
-		)
+	(label "BIN6_DT" (at 241.3 58.42 0)
+		(effects (font (size 3.5 3.5)) (justify left))
 	)
 	(wire (pts (xy 236.22 63.5) (xy 241.3 63.5))
@@
 		(stroke (width 0.254) (type default))
 	)
-	(global_label "BIN7_DT" (shape output) (at 327.66 58.42 0)
-		(effects (font (size 3.5 3.5)) (justify left))
-		(property "Intersheetrefs" "${INTERSHEET_REFS}" (at 327.66 58.42 0)
-			(effects (font (size 1.27 1.27)) (hide yes))
-		)
+	(label "BIN7_DT" (at 327.66 58.42 0)
+		(effects (font (size 3.5 3.5)) (justify left))
 	)
 	(wire (pts (xy 322.58 63.5) (xy 327.66 63.5))
@@
 		(stroke (width 0.254) (type default))
 	)
-	(global_label "BIN0_DT" (shape input) (at 162.56 107.95 180)
+	(label "BIN0_DT" (at 162.56 107.95 0)
 		(effects (font (size 3.5 3.5)) (justify right))
-		(property "Intersheetrefs" "${INTERSHEET_REFS}" (at 162.56 107.95 0)
-			(effects (font (size 1.27 1.27)) (hide yes))
-		)
 	)
 	(wire (pts (xy 167.64 113.03) (xy 162.56 113.03))
 		(stroke (width 0.254) (type default))
 	)
-	(global_label "BIN1_DT" (shape input) (at 162.56 113.03 180)
+	(label "BIN1_DT" (at 162.56 113.03 0)
 		(effects (font (size 3.5 3.5)) (justify right))
-		(property "Intersheetrefs" "${INTERSHEET_REFS}" (at 162.56 113.03 0)
-			(effects (font (size 1.27 1.27)) (hide yes))
-		)
 	)
 	(wire (pts (xy 167.64 118.11) (xy 162.56 118.11))
 		(stroke (width 0.254) (type default))
 	)
-	(global_label "BIN4_DT" (shape input) (at 162.56 118.11 180)
+	(label "BIN4_DT" (at 162.56 118.11 0)
 		(effects (font (size 3.5 3.5)) (justify right))
-		(property "Intersheetrefs" "${INTERSHEET_REFS}" (at 162.56 118.11 0)
-			(effects (font (size 1.27 1.27)) (hide yes))
-		)
 	)
 	(wire (pts (xy 167.64 123.19) (xy 162.56 123.19))
 		(stroke (width 0.254) (type default))
 	)
-	(global_label "BIN5_DT" (shape input) (at 162.56 123.19 180)
+	(label "BIN5_DT" (at 162.56 123.19 0)
 		(effects (font (size 3.5 3.5)) (justify right))
-		(property "Intersheetrefs" "${INTERSHEET_REFS}" (at 162.56 123.19 0)
-			(effects (font (size 1.27 1.27)) (hide yes))
-		)
 	)
 	(wire (pts (xy 167.64 128.27) (xy 162.56 128.27))
 		(stroke (width 0.254) (type default))
 	)
-	(global_label "BIN7_DT" (shape input) (at 162.56 128.27 180)
+	(label "BIN7_DT" (at 162.56 128.27 0)
 		(effects (font (size 3.5 3.5)) (justify right))
-		(property "Intersheetrefs" "${INTERSHEET_REFS}" (at 162.56 128.27 0)
-			(effects (font (size 1.27 1.27)) (hide yes))
-		)
 	)
 	(wire (pts (xy 167.64 133.35) (xy 162.56 133.35))
 		(stroke (width 0.254) (type default))
 	)
-	(global_label "BIN6_DT" (shape input) (at 162.56 133.35 180)
+	(label "BIN6_DT" (at 162.56 133.35 0)
 		(effects (font (size 3.5 3.5)) (justify right))
-		(property "Intersheetrefs" "${INTERSHEET_REFS}" (at 162.56 133.35 0)
-			(effects (font (size 1.27 1.27)) (hide yes))
-		)
 	)
 	(wire (pts (xy 167.64 138.43) (xy 162.56 138.43))
 		(stroke (width 0.254) (type default))
 	)
-	(global_label "BIN3_DT" (shape input) (at 162.56 138.43 180)
+	(label "BIN3_DT" (at 162.56 138.43 0)
 		(effects (font (size 3.5 3.5)) (justify right))
-		(property "Intersheetrefs" "${INTERSHEET_REFS}" (at 162.56 138.43 0)
-			(effects (font (size 1.27 1.27)) (hide yes))
-		)
 	)
 	(wire (pts (xy 167.64 143.51) (xy 162.56 143.51))
 		(stroke (width 0.254) (type default))
 	)
-	(global_label "BIN2_DT" (shape input) (at 162.56 143.51 180)
+	(label "BIN2_DT" (at 162.56 143.51 0)
 		(effects (font (size 3.5 3.5)) (justify right))
-		(property "Intersheetrefs" "${INTERSHEET_REFS}" (at 162.56 143.51 0)
-			(effects (font (size 1.27 1.27)) (hide yes))
-		)
 	)
 	(wire (pts (xy 254 107.95) (xy 259.08 107.95))
@@
 		(stroke (width 0.254) (type default))
 	)
-	(global_label "USB to host" (shape bidirectional) (at 259.08 143.51 0)
-		(effects (font (size 3.5 3.5)) (justify left))
-		(property "Intersheetrefs" "${INTERSHEET_REFS}" (at 259.08 143.51 0)
-			(effects (font (size 1.27 1.27)) (hide yes))
-		)
+	(label "USB to host" (at 259.08 143.51 0)
+		(effects (font (size 3.5 3.5)) (justify left))
 	)
 	(text "Load cell wires: red E+, black E-, green A+, white A-. Check against your own cell."
